File: Hardware/Head/Projet_Animatronic.kicad_sch (KiCad schematic)
At the start: 25 parts, among them J101 Conn_01x15, J102 Conn_01x04, J103 Conn_01x04, J104 Conn_01x06, J105 Conn_01x06, J106 Conn_01x06, U101 PCA9685PW

Commit message: maj PCB
Parts:
- removed C101: 100n, Capacitor_SMD:C_0402_1005Metric, symbol Device:C_Small
- removed J102, J103: Conn_01x04, Connector_JST:JST_XH_B4B-XH-A_1x04_P2.50mm_Vertical, symbol Connector_Generic:Conn_01x04
- removed U101: PCA9685PW, Package_SO:TSSOP-28_4.4x9.7mm_P0.65mm, symbol Driver_LED:PCA9685PW
- removed U2, U3, U4, U5: ~, buck:173010x42, symbol buck:173010x42
- added J1: Conn_01x04, symbol Connector_Generic:Conn_01x04
Connections:
- net +5V: now also J1.1 (Pin_1)
- net GND: now also J1.4 (Pin_4)
- net I2C_SCL: now also J1.3 (Pin_3)
- net I2C_SDA: now also J1.2 (Pin_2)
- net PWM_TIM1_CH1: now also J101.7 (Pin_7); no longer J101.2 (Pin_2)
- net PWM_TIM1_CH2: now also J101.6 (Pin_6); no longer J101.3 (Pin_3)
- net PWM_TIM1_CH3: now also J101.5 (Pin_5); no longer J101.4 (Pin_4)
- net PWM_TIM1_CH4: now also J101.4 (Pin_4); no longer J101.5 (Pin_5)
- net PWM_TIM2_CH1: now also J101.3 (Pin_3); no longer J101.6 (Pin_6)
- net PWM_TIM2_CH2: now also J101.2 (Pin_2); no longer J101.7 (Pin_7)
- no-connect marks 10 -> 0
Other:
- note removed: "LED"
- moved on the sheet: U6, U7
