File: Hardware/Body/ProjetCorps.kicad_pcb (KiCad board)
At the start: 4 copper layers, 60 x 58 mm, 65 parts, among them J101 Conn_01x02, J102 Conn_01x03, J103 Conn_01x03, J104 Conn_01x15, J105 Conn_ST_STDC14, SW101 SW_SPDT, SW102 SW_SPST, SW201 SW_SPST, SW301 SW_SPST, SW401 SW_SPST, SW501 SW_SPST, SW601 SW_SPST, SW701 SW_SPST, SW801 SW_SPST, U1 STM32L476RGTx, U101 STM32L412KBTx, U103 AZ1117-3.3, U104 173010542

Commit message: maj PCB
Parts:
- removed C105: 100n, Capacitor_SMD:C_0402_1005Metric
- removed C201, C301, C401, C501, C601, C701: 10n, Capacitor_SMD:C_0402_1005Metric
- removed R106: 100k, Resistor_SMD:R_0402_1005Metric
- removed R201, R202, R301, R302, R401, R402, R501, R502, R601, R602, R701, R702: 10k, Resistor_SMD:R_0402_1005Metric
- removed SW102, SW201, SW301, SW401, SW501, SW601, SW701: SW_SPST, Button_Switch_SMD:SW_Push_1P1T_NO_6x6mm_H9.5mm
- removed U101: STM32L412KBTx, Package_QFP:LQFP-32_7x7mm_P0.8mm
- added J1: Conn_01x04, Connector_JST:JST_EH_B4B-EH-A_1x04_P2.50mm_Vertical, F.Cu at (234.1, 62.3)
- added J2: Conn_01x06, Connector_JST:JST_EH_B6B-EH-A_1x06_P2.50mm_Vertical, F.Cu at (180.7, 96.0)
- added J3: Conn_01x04, Connector_JST:JST_EH_B4B-EH-A_1x04_P2.50mm_Vertical, F.Cu at (194.6, 96.1)
- C104: value 100n -> 400n
- U1: value STM32L476RGTx -> STM32G474RETx
- moved U1 201.6 mm to (199.2, 66.7), turned to -90 degrees
- moved R102 85.6 mm to (211.8, 66.6)
- moved C102 81.0 mm to (211.1, 74.0)
- moved C104 81.0 mm to (213.8, 74.5)
- moved J105 79.8 mm to (190.5, 83.7), turned to -90 degrees
- moved C101 78.8 mm to (216.1, 66.3)
- moved C103 78.8 mm to (215.1, 66.3)
- moved R101 77.2 mm to (215.8, 70.7)
- moved C107 73.7 mm to (213.1, 85.1)
- moved J101 73.7 mm to (222.7, 94.8)
- moved SW101 73.7 mm to (204.0, 94.8)
- moved U103 73.7 mm to (219.7, 85.1)
- moved U104 73.7 mm to (204.0, 89.0)
- moved H104 73.4 mm to (233.3, 101.3)
- moved H102 71.6 mm to (231.5, 52.6)
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Connections:
- C801 pad 1: BTN_7 -> BTN_1
- J104 pad 2: PWM_TIM1_CH1 -> PWM_TIM2_CH2
- J104 pad 3: PWM_TIM1_CH2 -> PWM_TIM2_CH1
- J104 pad 4: PWM_TIM1_CH3 -> PWM_TIM1_CH4
- J104 pad 5: PWM_TIM1_CH4 -> PWM_TIM1_CH3
- J104 pad 6: PWM_TIM2_CH1 -> PWM_TIM1_CH2
- J104 pad 7: PWM_TIM2_CH2 -> PWM_TIM1_CH1
- R801 pad 2: BTN_7 -> BTN_1
- U1 pad 1: unconnected-(U1-VBAT-Pad1) -> +3.3V
- U1 pad 10: unconnected-(U1-PC2-Pad10) -> PWM_TIM1_CH3
- U1 pad 11: unconnected-(U1-PC3-Pad11) -> PWM_TIM1_CH4
- U1 pad 12: unconnected-(U1-VSSA-Pad12) -> PWM_TIM2_CH1
- U1 pad 13: unconnected-(U1-VDDA-Pad13) -> PWM_TIM2_CH2
- U1 pad 14: unconnected-(U1-PA0-Pad14) -> UART_DEBUG_TX
- U1 pad 15: unconnected-(U1-PA1-Pad15) -> GND
- U1 pad 16: unconnected-(U1-PA2-Pad16) -> +3.3V
- U1 pad 17: unconnected-(U1-PA3-Pad17) -> UART_DEBUG_RX
- U1 pad 18: Net-(U1-VSS-Pad18) -> unconnected-(U1-PA4-Pad18)
- U1 pad 22: unconnected-(U1-PA6-Pad22) -> UART_HD_XL430
- U1 pad 25: unconnected-(U1-PC5-Pad25) -> BTN_1
- U1 pad 27: unconnected-(U1-PB1-Pad27) -> GND
- U1 pad 28: unconnected-(U1-PB2-Pad28) -> +3.3V
- U1 pad 29: unconnected-(U1-PB10-Pad29) -> +3.3V
- U1 pad 30: unconnected-(U1-PB11-Pad30) -> UART_hc05_RX
- U1 pad 31: Net-(U1-VSS-Pad18) -> GND
- U1 pad 32: unconnected-(U1-VDD-Pad32) -> +3.3V
- U1 pad 33: unconnected-(U1-PB12-Pad33) -> UART_hc05_TX
- U1 pad 42: UART_DEBUG_TX -> PWM_TIM2_CH3
- U1 pad 43: UART_DEBUG_RX -> unconnected-(U1-PA9-Pad43)
- U1 pad 44: unconnected-(U1-PA11-Pad44) -> PWM_TIM2_CH4
- U1 pad 45: unconnected-(U1-PA12-Pad45) -> SWDIO
- U1 pad 46: SWDIO -> SWCLK
- U1 pad 47: Net-(U1-VSS-Pad18) -> GND
- U1 pad 48: unconnected-(U1-VDDUSB-Pad48) -> +3.3V
- U1 pad 49: SWCLK -> I2C_SCL
- U1 pad 50: unconnected-(U1-PA15-Pad50) -> I2C_SDA
- U1 pad 52: unconnected-(U1-PC11-Pad52) -> UART_mp3_TX
- U1 pad 53: unconnected-(U1-PC12-Pad53) -> UART_mp3_RX
- U1 pad 57: unconnected-(U1-PB5-Pad57) -> LED1
- U1 pad 58: unconnected-(U1-PB6-Pad58) -> LED2
- U1 pad 59: I2C_SCL -> LED3
- U1 pad 61: I2C_SDA -> unconnected-(U1-PB8-Pad61)
- U1 pad 63: Net-(U1-VSS-Pad18) -> GND
- U1 pad 64: unconnected-(U1-VDD-Pad64) -> +3.3V
- U1 pad 7: NRST -> unconnected-(U1-PG10-Pad7)
- U1 pad 8: unconnected-(U1-PC0-Pad8) -> PWM_TIM1_CH1
- U1 pad 9: unconnected-(U1-PC1-Pad9) -> PWM_TIM1_CH2
Routing:
- net +3.3V: track 48.7 -> 0.00 mm, vias 20 -> 0
- net UART_HD_XL430: track 44.8 -> 0.00 mm, vias 2 -> 0
- net BTN_7: track 40.5 -> 0.00 mm, vias 2 -> 0
- net UART_DEBUG_RX: track 32.9 -> 0.00 mm
- net UART_DEBUG_TX: track 28.1 -> 0.00 mm
- net SWDIO: track 27.7 -> 0.00 mm, vias 2 -> 0
- net SWCLK: track 26.4 -> 0.00 mm, vias 2 -> 0
- net NRST: track 26.2 -> 0.00 mm, vias 2 -> 0
- net I2C_SDA: track 23.6 -> 0.00 mm, vias 1 -> 0
- net BTN_6: track 23.2 -> 0.00 mm
- net BTN_4: track 21.6 -> 0.00 mm
- net I2C_SCL: track 20.7 -> 0.00 mm, vias 1 -> 0
- net BTN_2: track 20.4 -> 0.00 mm
- net +5V: track 17.7 -> 0.00 mm, vias 4 -> 0
- net Net-(SW401-A): track 10.8 -> 0.00 mm
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- removed copper zone on In1.Cu, net +12V
- removed copper zone on In1.Cu, net +3.3V
- removed copper zone on F.Cu, net +5V
- removed copper zone on In1.Cu, net +5V
- removed copper zone on B.Cu, net GND
- removed copper zone on F.Cu, net GND
- removed copper zone on In2.Cu, net GND
- removed copper zone on In1.Cu, net Net-(J101-Pin_2)
Other:
- board outline removed
- board text removed: "1"
- board text removed: "12V 5V 3V3"
- board text removed: "BTN 1|2 3|4 5|6 X|7"
- board text removed: "LED 1 LED 2 LED 3"
- board text removed: "NRST"
- board text removed: "XL430"

Commit message: update pcb body
Parts:
- added C1: 100n, Capacitor_SMD:C_0402_1005Metric, F.Cu at (82.9, 63.2)
- added SW1: SW_SPST, Button_Switch_SMD:SW_Push_1P1T_NO_6x6mm_H9.5mm, F.Cu at (85.2, 70.2)
- moved SW801 173.4 mm to (51.6, 82.1), turned to -90 degrees
- moved C801 169.7 mm to (49.6, 76.6), turned to 180 degrees
- moved R801 167.9 mm to (51.5, 76.6), turned to 180 degrees
- moved R802 166.0 mm to (53.4, 76.6), turned to 180 degrees
- moved C103 156.7 mm to (59.0, 79.0)
- moved C101 155.5 mm to (61.2, 79.0)
- moved C104 151.6 mm to (62.3, 79.0)
- moved R101 151.1 mm to (65.0, 79.6), turned to 90 degrees
- moved C102 151.0 mm to (60.1, 79.0), turned to -90 degrees
- moved J3 150.9 mm to (44.1, 84.6), turned to 90 degrees
- moved R102 146.2 mm to (66.2, 79.6), turned to 90 degrees
- moved C107 142.2 mm to (70.9, 83.7)
- moved J101 142.2 mm to (80.5, 93.3)
- moved SW101 142.2 mm to (61.8, 93.3)
- moved U103 142.2 mm to (77.5, 83.7)
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Connections:
- U1 pad 30: UART_hc05_RX -> UART_hc05_TX
- U1 pad 33: UART_hc05_TX -> UART_hc05_RX
- U1 pad 40: unconnected-(U1-PC8-Pad40) -> I2C_SCL
- U1 pad 41: unconnected-(U1-PC9-Pad41) -> I2C_SDA
- U1 pad 42: PWM_TIM2_CH3 -> unconnected-(U1-PA8-Pad42)
- U1 pad 45: SWDIO -> unconnected-(U1-PA11-Pad45)
- U1 pad 46: SWCLK -> unconnected-(U1-PA12-Pad46)
- U1 pad 49: I2C_SCL -> SWDIO
- U1 pad 50: I2C_SDA -> SWCLK
- U1 pad 7: unconnected-(U1-PG10-Pad7) -> NRST
Routing:
- net +5V: track 0.00 -> 66.2 mm, vias 0 -> 2
- net +3.3V: track 0.00 -> 45.9 mm, vias 0 -> 9
- net PWM_TIM2_CH4: track 0.00 -> 44.3 mm, vias 0 -> 1
- net I2C_SDA: track 0.00 -> 41.9 mm, vias 0 -> 1
- net I2C_SCL: track 0.00 -> 41.3 mm, vias 0 -> 1
- net UART_hc05_TX: track 0.00 -> 40.5 mm, vias 0 -> 1
- net UART_HD_XL430: track 0.00 -> 36.1 mm
- net UART_hc05_RX: track 0.00 -> 34.9 mm, vias 0 -> 1
- net UART_DEBUG_RX: track 0.00 -> 33.8 mm, vias 0 -> 2
- net NRST: track 0.00 -> 30.3 mm, vias 0 -> 2
- net UART_DEBUG_TX: track 0.00 -> 29.3 mm, vias 0 -> 2
- net UART_mp3_RX: track 0.00 -> 26.8 mm, vias 0 -> 2
- net UART_mp3_TX: track 0.00 -> 25.5 mm, vias 0 -> 1
- net BTN_1: track 0.00 -> 16.9 mm
- net LED3: track 0.00 -> 15.7 mm
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- added copper zone on In1.Cu, net +12V
- added copper zone on In1.Cu, net +3.3V
- added copper zone on In1.Cu, net +5V
- added copper zone on B.Cu, net GND
- added copper zone on F.Cu, net GND
- added copper zone on In2.Cu, net GND
- added copper zone on In1.Cu, net Net-(J101-Pin_2)
Other:
- board outline added: 60 x 60 mm
- board text added: "3V3 5V 12V"
- board text added: "BTN"
- board text added: "C101"
- board text added: "C102"
- board text added: "C103"
- board text added: "C104"
- board text added: "C107"
- board text added: "C801"
- board text added: "J101"
- board text added: "J102"
- board text added: "J103"
- board text added: "J105"
- board text added: "LED"
- board text added: "LED 1 LED 2 LED 3"
- board text added: "NRST"
- board text added: "R101"
- board text added: "R102"
- board text added: "R103"
- board text added: "R104"
- board text added: "R105"
- board text added: "R801"
- board text added: "R802"
- board text added: "SW101"
- board text added: "SW801"
- board text added: "U103"
- board text added: "U104"
- board text added: "XL430"

Commit message: check Fiack
Parts:
- added C2: 100n, Capacitor_SMD:C_0402_1005Metric, F.Cu at (66.5, 62.6)
- added C3: 10n, Capacitor_SMD:C_0402_1005Metric, F.Cu at (62.1, 72.0)
- added C4: 1u, Capacitor_SMD:C_0402_1005Metric, F.Cu at (60.1, 72.0)
- added C5: 100n, Capacitor_SMD:C_0402_1005Metric, F.Cu at (62.1, 70.9)
- added C6: 1u, Capacitor_SMD:C_0402_1005Metric, F.Cu at (60.1, 70.9)
- C104: value 400n -> 100n
- moved C103 22.2 mm to (77.4, 66.6)
- moved R101 21.5 mm to (63.2, 58.2), turned to 0 degrees
- moved R102 21.4 mm to (65.2, 58.2), turned to 180 degrees
- moved C101 18.4 mm to (66.5, 61.4), turned to 0 degrees
- moved C102 13.5 mm to (73.5, 77.4), turned to 180 degrees
- moved C1 11.0 mm to (72.0, 62.0)
- moved C104 5.49 mm to (62.6, 73.5), turned to 90 degrees
- moved C106 1.64 mm to (81.7, 86.3)
Routing:
- net +5V: track 66.2 -> 105.4 mm, vias 2 -> 3
- net GND: track 0.00 -> 29.4 mm, vias 112 -> 136
- net +3.3V: track 45.9 -> 31.9 mm, vias 9 -> 16
- net PWM_TIM2_CH4: track 44.3 -> 33.4 mm
- net I2C_SDA: track 41.9 -> 33.9 mm
- net I2C_SCL: track 41.3 -> 33.4 mm
- net UART_hc05_TX: track 40.5 -> 36.8 mm
- net UART_DEBUG_TX: track 29.3 -> 25.9 mm
- net UART_DEBUG_RX: track 33.8 -> 31.0 mm
- net UART_hc05_RX: track 34.9 -> 32.9 mm
- net UART_HD_XL430: track 36.1 -> 34.4 mm
- net LED3: track 15.7 -> 16.7 mm
- net LED2: track 15.3 -> 15.9 mm
- net NRST: track 30.3 -> 29.8 mm

Commit message: update pcb body
Connections:
- J3 pad 3: PWM_TIM2_CH4 -> PWM_TIM4_CH1
- U1 pad 44: PWM_TIM2_CH4 -> unconnected-(U1-PA10-Pad44)
- U1 pad 45: unconnected-(U1-PA11-Pad45) -> PWM_TIM4_CH1
Routing:
- net PWM_TIM2_CH4: track 33.4 -> 0.00 mm, vias 1 -> 0
- net PWM_TIM4_CH1: track 0.00 -> 32.0 mm, vias 0 -> 1
- net GND: vias 136 -> 75
Other:
- board text added: "J2"

Commit message: update tof int
Connections:
- J104 pad 14: +12V -> TOF_INT
- U1 pad 39: unconnected-(U1-PC7-Pad39) -> TOF_INT
Routing:
- net TOF_INT: track 0.00 -> 31.5 mm, vias 0 -> 1
- net GND: vias 75 -> 76
