File: Hardware/Body/ProjetCorps.kicad_sch (KiCad schematic)
At the start: 38 parts, among them J1 Screw_Terminal_01x20, J101 Conn_01x02, J102 Conn_01x03, J103 Conn_01x03, J104 Conn_01x15, J105 Conn_ST_STDC14, J2 Screw_Terminal_01x20, SW101 SW_SPDT, SW102 SW_SPST, U1 STM32L476RGTx, U103 AZ1117-3.3, U104 173010542

Commit message: maj PCB
Parts:
- removed C105: 100n, Capacitor_SMD:C_0402_1005Metric, symbol Device:C_Small
- removed J1, J2: Screw_Terminal_01x20, symbol Connector:Screw_Terminal_01x20
- removed R106: 100k, Resistor_SMD:R_0402_1005Metric, symbol Device:R_Small
- removed SW102: SW_SPST, Button_Switch_SMD:SW_Push_1P1T_NO_6x6mm_H9.5mm, symbol Switch:SW_SPST
- removed U1: STM32L476RGTx, Package_QFP:LQFP-64_10x10mm_P0.5mm, symbol MCU_ST_STM32L4:STM32L476RGTx
- added J1, J3: Conn_01x04, Connector_JST:JST_EH_B4B-EH-A_1x04_P2.50mm_Vertical, symbol Connector_Generic:Conn_01x04
- added J2: Conn_01x06, Connector_JST:JST_EH_B6B-EH-A_1x06_P2.50mm_Vertical, symbol Connector_Generic:Conn_01x06
- added U1: STM32G474RETx, Package_QFP:LQFP-64_10x10mm_P0.5mm, symbol MCU_ST_STM32G4:STM32G474RETx
- C104: value 100n -> 400n
Connections:
- net +3.3V: now also U1.1 (VBAT), U1.16 (VDD), U1.28 (VREF+), U1.29 (VDDA), U1.32 (VDD), U1.48 (VDD), U1.64 (VDD)
- net +5V: now also J1.3 (Pin_3), J2.2 (Pin_2), J3.4 (Pin_4)
- net BTN_1: now also U1.25 (PB1)
- net GND: now also J1.4 (Pin_4), J2.3 (Pin_3), J3.2 (Pin_2), U1.15 (VSS), U1.27 (VSSA), U1.31 (VSS), U1.47 (VSS), U1.63 (VSS)
- net I2C_SCL: now also U1.49 (PA13)
- net I2C_SDA: now also U1.50 (PA14)
- net LED1: now also U1.57 (PB4)
- net LED2: now also U1.58 (PB5)
- net LED3: now also U1.59 (PB6)
- net PWM_TIM1_CH1: now also J104.7 (Pin_7), U1.8 (PC0); no longer J104.2 (Pin_2)
- net PWM_TIM1_CH2: now also J104.6 (Pin_6), U1.9 (PC1); no longer J104.3 (Pin_3)
- net PWM_TIM1_CH3: now also J104.5 (Pin_5), U1.10 (PC2); no longer J104.4 (Pin_4)
- net PWM_TIM1_CH4: now also J104.4 (Pin_4), U1.11 (PC3); no longer J104.5 (Pin_5)
- net PWM_TIM2_CH1: now also J104.3 (Pin_3), U1.12 (PA0); no longer J104.6 (Pin_6)
- net PWM_TIM2_CH2: now also J104.2 (Pin_2), U1.13 (PA1); no longer J104.7 (Pin_7)
- net SWCLK: now also U1.46 (PA12)
- net SWDIO: now also U1.45 (PA11)
- net UART_DEBUG_RX: now also U1.17 (PA3)
- net UART_DEBUG_TX: now also U1.14 (PA2)
- net UART_HD_XL430: now also U1.22 (PC4)
- new net PWM_TIM2_CH3: U1.42 (PA8)
- new net PWM_TIM2_CH4: J3.3 (Pin_3), U1.44 (PA10)
- new net UART_hc05_RX: J2.5 (Pin_5), U1.30 (PB10)
- new net UART_hc05_TX: J2.4 (Pin_4), U1.33 (PB11)
- new net UART_mp3_RX: J1.1 (Pin_1), U1.53 (PC11)
- new net UART_mp3_TX: J1.2 (Pin_2), U1.52 (PC10)
- no-connect marks 4 -> 36
Other:
- removed sheet button_2
- removed sheet button_3
- removed sheet button_4
- removed sheet button_5
- removed sheet button_6
- removed sheet button_7
- note added: "1:key 6:state"
- note added: "HCO5/bluetooth"
- note added: "LED"
- note added: "module mp3"
- moved on the sheet: C101, C102, C103, C104

Commit message: update pcb body
Parts:
- added C1: 100n, Capacitor_SMD:C_0402_1005Metric, symbol Device:C_Small
- added SW1: SW_SPST, Button_Switch_SMD:SW_Push_1P1T_NO_6x6mm_H9.5mm, symbol Switch:SW_SPST
Connections:
- net GND: now also C1.2, SW1.2 (B)
- net I2C_SCL: now also U1.40 (PC8); no longer U1.49 (PA13)
- net I2C_SDA: now also U1.41 (PC9); no longer U1.50 (PA14)
- net NRST: now also U1.7 (PG10), C1.1, SW1.1 (A)
- net SWCLK: now also U1.50 (PA14); no longer U1.46 (PA12)
- net SWDIO: now also U1.49 (PA13); no longer U1.45 (PA11)
- net UART_hc05_RX: now also U1.33 (PB11); no longer U1.30 (PB10)
- net UART_hc05_TX: now also U1.30 (PB10); no longer U1.33 (PB11)
- net PWM_TIM2_CH3: no longer names the net of U1.42 (PA8)
Other:
- note added: "4VDDx100n"
- note added: "DOUT"
- moved on the sheet: C101, C102, C103, C104

Commit message: check Fiack
Parts:
- added C2, C5: 100n, Capacitor_SMD:C_0402_1005Metric, symbol Device:C_Small
- added C3: 10n, Capacitor_SMD:C_0402_1005Metric, symbol Device:C_Small
- added C4, C6: 1u, Capacitor_SMD:C_0402_1005Metric, symbol Device:C_Small
- C104: value 400n -> 100n
Connections:
- net +3.3V: now also C2.1, C3.1, C4.1, C5.2, C6.2
- net GND: now also C2.2, C3.2, C4.2, C5.1, C6.1
Other:
- moved on the sheet: C1, C101, C102, C103, C104, SW1, U1

Commit message: update pcb body
Connections:
- net PWM_TIM4_CH1: now reaches U1.45 (PA11)
- net PWM_TIM4_CH1: now also J3.3 (Pin_3)
- net PWM_TIM2_CH4: no longer names the net of U1.44 (PA10)
- net PWM_TIM2_CH4: no longer J3.3 (Pin_3)
Changed lines of the file:
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@@
 	)
 	(no_connect
+		(at 146.05 123.19)
+	)
+	(no_connect
 		(at 220.98 41.91)
 	)
@@
 	)
 	(no_connect
-		(at 146.05 125.73)
-	)
-	(no_connect
 		(at 146.05 173.99)
 	)
@@
 		)
 	)
-	(wire
-		(pts
-			(xy 146.05 123.19) (xy 148.59 123.19)
-		)
-		(stroke
-			(width 0)
-			(type default)
-		)
-	)
 	(polyline
 		(pts
@@
 	(wire
 		(pts
+			(xy 146.05 125.73) (xy 148.59 125.73)
+		)
+		(stroke
+			(width 0)
+			(type default)
+		)
+	)
+	(wire
+		(pts
 			(xy 146.05 133.35) (xy 148.59 133.35)
 		)
@@
 		)
 	)
-	(global_label "PWM_TIM2_CH4"
+	(global_label "PWM_TIM4_CH1"
 		(shape input)
 		(at 124.46 52.07 180)
@@
 		)
 	)
-	(global_label "PWM_TIM2_CH4"
+	(global_label "PWM_TIM4_CH1"
 		(shape input)
-		(at 148.59 123.19 0)
+		(at 148.59 125.73 0)
 		(fields_autoplaced yes)
 		(effects
@@
 		)
 		(property "Intersheetrefs" "${INTERSHEET_REFS}"
-			(at 165.7265 123.19 0)
+			(at 165.7265 125.73 0)
 			(effects
 				(font
@@
 		)
 		(instances
-			(project ""
+			(project "ProjetCorps"
 				(path "/72512375-e259-4361-868e-851dab973787"
 					(reference "#PWR09")

Commit message: update tof int
Connections:
- net +12V: no longer J104.14 (Pin_14)
- net TOF_INT: now reaches U1.39 (PC7)
- net TOF_INT: now also J104.14 (Pin_14)
- no-connect marks 36 -> 35
Changed lines of the file:
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@@
 	)
 	(no_connect
-		(at 110.49 138.43)
-	)
-	(no_connect
 		(at 110.49 153.67)
 	)
@@
 	(wire
 		(pts
+			(xy 104.14 138.43) (xy 110.49 138.43)
+		)
+		(stroke
+			(width 0)
+			(type default)
+		)
+	)
+	(wire
+		(pts
 			(xy 135.89 83.82) (xy 135.89 91.44)
 		)
@@
 		)
 	)
+	(global_label "TOF_INT"
+		(shape input)
+		(at 104.14 138.43 180)
+		(fields_autoplaced yes)
+		(effects
+			(font
+				(size 1.27 1.27)
+			)
+			(justify right)
+		)
+		(property "Intersheetrefs" "${INTERSHEET_REFS}"
+			(at 93.8976 138.43 0)
+			(effects
+				(font
+					(size 1.27 1.27)
+				)
+				(justify right)
+				(hide yes)
+			)
+		)
+	)
 	(global_label "BTN_1"
 		(shape input)
@@
 		)
 	)
+	(global_label "TOF_INT"
+		(shape input)
+		(at 97.79 33.02 180)
+		(fields_autoplaced yes)
+		(effects
+			(font
+				(size 1.27 1.27)
+			)
+			(justify right)
+		)
+		(property "Intersheetrefs" "${INTERSHEET_REFS}"
+			(at 87.5476 33.02 0)
+			(effects
+				(font
+					(size 1.27 1.27)
+				)
+				(justify right)
+				(hide yes)
+			)
+		)
+	)
 	(global_label "PWM_TIM1_CH4"
 		(shape input)
@@
 					(unit 1)
 				)
-			)
-		)
-	)
-	(symbol
-		(lib_id "power:+12V")
-		(at 97.79 33.02 90)
-		(unit 1)
-		(exclude_from_sim no)
-		(in_bom yes)
-		(on_board yes)
-		(dnp no)
-		(fields_autoplaced yes)
-		(property "Reference" "#PWR0114"
-			(at 101.6 33.02 0)
-			(effects
-				(font
-					(size 1.27 1.27)
-				)
-				(hide yes)
-			)
-		)
-		(property "Value" "+12V"
-			(at 93.98 33.0199 90)
-			(effects
-				(font
-					(size 1.27 1.27)
-				)
-				(justify left)
-			)
-		)
-		(property "Footprint" ""
-			(at 97.79 33.02 0)
-			(effects
-				(font
-					(size 1.27 1.27)
-				)
-				(hide yes)
-			)
-		)
-		(property "Datasheet" ""
-			(at 97.79 33.02 0)
-			(effects
-				(font
-					(size 1.27 1.27)
-				)
-				(hide yes)
-			)
-		)
-		(property "Description" "Power symbol creates a global label with name \"+12V\""
-			(at 97.79 33.02 0)
-			(effects
-				(font
-					(size 1.27 1.27)
-				)
-				(hide yes)
-			)
-		)
-		(pin "1"
-		)
-		(instances
-			(project "ProjetCorps"
-				(path "/72512375-e259-4361-868e-851dab973787"
-					(reference "#PWR0114")
-					(unit 1)
-				)
