File: Hardware/pcb/Body/ProjetCorps.kicad_pcb (KiCad board)
At the start: 4 copper layers, 60 x 60 mm, 47 parts, among them J1 Conn_01x04, J101 Conn_01x02, J102 Conn_01x03, J103 Conn_01x03, J104 Conn_01x15, J105 Conn_ST_STDC14, J2 Conn_01x06, J3 Conn_01x04, SW1 SW_SPST, SW101 SW_SPDT, SW801 SW_SPST, U1 STM32G474RETx, U103 AZ1117-3.3, U104 173010542

Commit message: pcb body & gant maj
Parts:
- added R1: 100k, Resistor_SMD:R_0805_2012Metric, F.Cu at (59.0, 64.8)
Routing:
- net UART_HD_XL430: track 34.4 -> 36.0 mm

Commit message: PCB body & gant V3
Parts:
- moved R1 0.98 mm to (58.0, 65.0), turned to -90 degrees
Routing:
- net UART_HD_XL430: track 36.0 -> 34.6 mm
