File: Hardware/pcb/Gant/PCB_Gant/PCB_Gant.kicad_pcb (KiCad board)
At the start: 4 copper layers, 42 x 40 mm, 34 parts, among them J1 Conn_ST_STDC14, J2 Conn_01x06, SW1 SW_SPST, SW2 RotaryEncoder, U1 STM32G431KBTx, U2 MCP602, U3 MCP602, U5 AZ1117-3.3

Commit message: pcb body & gant maj
Parts:
- added C10: 100n, Capacitor_SMD:C_0402_1005Metric, F.Cu at (104.7, 73.1)
- added C11: 100n, Capacitor_SMD:C_0402_1005Metric, F.Cu at (119.7, 70.8)
- added C12: 100n, Capacitor_SMD:C_0402_1005Metric, F.Cu at (127.8, 79.5)
- added C9: 100n, Capacitor_SMD:C_0402_1005Metric, F.Cu at (112.0, 81.0)
- added J3: Conn_01x02, Connector_JST:JST_EH_B2B-EH-A_1x02_P2.50mm_Vertical, F.Cu at (133.2, 79.3)
- moved J1 1.22 mm to (129.0, 87.3)
- moved R6 0.90 mm to (116.0, 67.2)
- moved R4 0.54 mm to (107.6, 67.8), turned to 10 degrees
- moved R10 0.50 mm to (124.4, 67.8), turned to -10 degrees
Connections:
- U2 pad 4: GND -> Net-(U2C-V-)
- U2 pad 8: +3.3V -> Net-(U2C-V+)
- U3 pad 4: GND -> Net-(U3C-V-)
- U3 pad 8: +3.3V -> Net-(U3C-V+)
Routing:
- net Net-(U2C-V+): track 0.00 -> 3.51 mm, vias 0 -> 2
- net Net-(U3C-V-): track 0.00 -> 3.41 mm
- net Net-(U3C-V+): track 0.00 -> 2.15 mm, vias 0 -> 1
- net Net-(U2C-V-): track 0.00 -> 1.45 mm
- net UART2_DEBUG_RX: track 24.2 -> 22.9 mm
- net SWCLK: track 8.15 -> 6.94 mm
- net SWDIO: track 10.5 -> 9.27 mm
- net Net-(U3A-+): track 6.92 -> 8.03 mm
- net Net-(U2B-+): track 16.0 -> 16.9 mm

Commit message: PCB body & gant V3
Parts:
- removed C10, C11: 100n, Capacitor_SMD:C_0402_1005Metric
- removed SW1: SW_SPST, Button_Switch_THT:SW_PUSH_6mm_H9.5mm
- added Flex1neg1: TestPoint, TestPoint:TestPoint_Pad_D1.5mm, F.Cu at (111.6, 72.8)
- added Flex1pos1: TestPoint, TestPoint:TestPoint_Pad_D1.5mm, F.Cu at (99.5, 75.6)
- added Flex2neg1: TestPoint, TestPoint:TestPoint_Pad_D1.5mm, F.Cu at (99.5, 79.2)
- added Flex2pos1: TestPoint, TestPoint:TestPoint_Pad_D1.5mm, F.Cu at (114.7, 71.6)
- added Flex3neg1: TestPoint, TestPoint:TestPoint_Pad_D1.5mm, F.Cu at (118.5, 75.3)
- added Flex3pos1: TestPoint, TestPoint:TestPoint_Pad_D1.5mm, F.Cu at (119.4, 71.8)
- moved C6 14.4 mm to (113.4, 90.3), turned to 135 degrees
- moved C3 3.74 mm to (111.9, 87.5), turned to 90 degrees
- moved C9 3.65 mm to (110.1, 77.9)
- moved C12 1.66 mm to (127.3, 77.9)
- moved C4 1.43 mm to (123.8, 80.7), turned to -45 degrees
- moved C1 1.38 mm to (111.9, 89.5), turned to -90 degrees
- moved R5 1.20 mm to (102.9, 76.9)
- moved R7 1.20 mm to (102.9, 79.1)
- moved R8 1.20 mm to (102.9, 78.0)
- moved U2 1.20 mm to (106.8, 75.9)
- moved C5 0.96 mm to (122.5, 81.3), turned to -45 degrees
Connections:
- C12 pad 2: Net-(U3C-V+) -> GND
- C9 pad 1: Net-(U2C-V+) -> GND
- R13 pad 1: +5V -> +3.3V
- R14 pad 1: +5V -> +3.3V
- U2 pad 4: Net-(U2C-V-) -> GND
- U2 pad 8: Net-(U2C-V+) -> +3.3V
- U3 pad 4: Net-(U3C-V-) -> GND
- U3 pad 5: (no net) -> GND
- U3 pad 6: (no net) -> GND
- U3 pad 7: (no net) -> unconnected-(U3-Pad7)
- U3 pad 8: Net-(U3C-V+) -> +3.3V
Routing:
- net GND: track 6.51 -> 26.8 mm, vias 4 -> 47
- net NRST: track 22.2 -> 13.3 mm
- net Net-(U2A-+): track 6.70 -> 14.9 mm
- net Net-(U3A--): track 3.13 -> 10.8 mm
- net UART2_DEBUG_RX: track 22.9 -> 17.9 mm
- net Net-(U2B--): track 5.10 -> 10.0 mm
- net Net-(U2B-+): track 16.9 -> 21.1 mm
- net UART2_DEBUG_TX: track 16.7 -> 12.7 mm
- net GPIO1: track 16.4 -> 12.7 mm, vias 2 -> 0
- net Net-(U2A--): track 3.02 -> 6.68 mm
- net Net-(U2C-V+): track 3.51 -> 0.00 mm, vias 2 -> 0
- net Net-(U3C-V-): track 3.41 -> 0.00 mm
- net Net-(U3A-+): track 8.03 -> 11.0 mm
- net +5V: track 10.5 -> 7.91 mm, vias 5 -> 4
- net Net-(U3C-V+): track 2.15 -> 0.00 mm, vias 1 -> 0
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