File: Hardware/pcb/Gant/PCB_Gant/PCB_Gant.kicad_sch (KiCad schematic)
At the start: 4 parts, among them SW1 SW_SPST, U1 STM32G431KBTx

Commit message: modifications on schematic
Parts:
- added C3: 10n, symbol Device:C_Small
- added C4: 4u7, symbol Device:C_Small
- added C5, C6: 100n, symbol Device:C_Small
- C1: value 100n -> 1u
Connections:
- net +3.3V: now also U1.1 (VDD), U1.15 (VDDA), U1.17 (VDD), C3.1, C4.1, C5.1, C6.1
- net GND: now also C3.2, C4.2, C5.2, C6.2; no longer U1.1 (VDD), U1.15 (VDDA), U1.17 (VDD)
- net UART1_RX renamed UART2_DEBUG_RX
- net UART1_TX renamed UART2_DEBUG_TX
- net UART2_RX renamed UART1_HC05_RX
- net UART2_TX renamed UART1_HC05_TX

Commit message: PCB gant v1
Parts:
- added C7: 10u, Capacitor_SMD:C_0402_1005Metric, symbol Device:C_Small
- added C8: 22u, Capacitor_SMD:C_Elec_5x5.4, symbol Device:C_Small
- added H1, H2, H3, H4: MountingHole_Pad, MountingHole:MountingHole_3.2mm_M3_Pad_Via, symbol Mechanical:MountingHole_Pad
- added J1: Conn_ST_STDC14, Connector_PinHeader_1.27mm:PinHeader_2x07_P1.27mm_Vertical_SMD, symbol Connector:Conn_ST_STDC14
- added J2: Conn_01x06, Connector_JST:JST_EH_B6B-EH-A_1x06_P2.50mm_Vertical, symbol Connector_Generic:Conn_01x06
- added R1, R12, R8: 100, Resistor_SMD:R_0402_1005Metric, symbol Device:R_Small
- added R10, R4, R6: 10k, Resistor_SMD:R_2512_6332Metric, symbol Device:R_Variable
- added R11, R2, R7: 200, Resistor_SMD:R_0402_1005Metric, symbol Device:R_Small
- added R13, R14: 10k, Resistor_SMD:R_0402_1005Metric, symbol Device:R_Small
- added R3, R5, R9: 4.7k, Resistor_SMD:R_0402_1005Metric, symbol Device:R_Small
- added SW2: RotaryEncoder, Rotary_Encoder:RotaryEncoder_Alps_EC12E_Vertical_H20mm, symbol Device:RotaryEncoder
- added U2, U3: MCP602, Package_SO:SOIC-8_3.9x4.9mm_P1.27mm, symbol Amplifier_Operational:MCP602
- added U5: AZ1117-3.3, Package_TO_SOT_SMD:SOT-223-3_TabPin2, symbol Regulator_Linear:AZ1117-3.3
- C1, C2, C3, C4, C5, C6: footprint (none) -> Capacitor_SMD:C_0402_1005Metric
Connections:
- net +3.3V: now also C8.1, J1.3 (VCC), U2.8 (V+), U3.8 (V+), U5.2 (VO)
- net GND: now also C7.2, C8.2, H1.1, H2.1, H3.1, H4.1, J1.11 (GNDDetect), J1.5 (GND), J1.7 (GND), J2.3 (Pin_3), R10.2, R11.2, R2.2, R4.2, R6.2, R7.2, SW2.C, U2.4 (V-), U3.4 (V-), U5.1 (GND)
- net GPIO1: now also U2.1
- net GPIO2: now also U2.7
- net GPIO3: now also U3.1
- net NRST: now also J1.12 (~{RST})
- net SWCLK: now also J1.6 (JCLK/SWCLK)
- net SWDIO: now also J1.4 (JTMS/SWDIO)
- net UART1_HC05_RX: now also J2.5 (Pin_5)
- net UART1_HC05_TX: now also J2.4 (Pin_4)
- net UART2_DEBUG_RX: now also J1.13 (VCP_RX)
- net UART2_DEBUG_TX: now also J1.14 (VCP_TX)
- net DT: now reaches U1.10 (PA5)
- net DT: now also R14.2, SW2.B
- net CLK: now reaches U1.11 (PA6)
- net CLK: now also R13.2, SW2.A
- new net: R3.2, R4.1, U2.3 (+)
- new net: R1.1, R2.1, U2.2 (-)
- new net: R10.1, R9.2, U3.3 (+)
- new net: R7.1, R8.1, U2.6 (-)
- new net: R5.2, R6.1, U2.5 (+)
- new net: R11.1, R12.1, U3.2 (-)
- new net +5V: C7.1, J2.2 (Pin_2), R1.2, R12.2, R13.1, R14.1, R3.1, R5.1, R8.2, R9.1, U5.3 (VI)
- no-connect marks 15 -> 19
Other:
- note added: "1:key 6:state"
- note added: "Buck"
- note added: "Flex1"
- note added: "Flex2"
- note added: "Flex3"
- note added: "HCO5/bluetooth"
- note added: "Sonde Debug"
- note added: "Trous de fixation"
- note added: "Volume"
- note added: "±30%"

Commit message: PCB gant V2
Parts:
- SW1: footprint Button_Switch_SMD:SW_Push_1P1T_NO_6x6mm_H9.5mm -> Button_Switch_THT:SW_PUSH_6mm_H9.5mm
Changed lines of the file:
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@@
 			)
 		)
-		(property "Datasheet" "~"
+		(property "Datasheet" "https://github.com/mael-lukas/2425_Projet2A_Animatronic/blob/main/Datasheets/Flex_Sensor_Datasheet_v2019a-3304101.pdf"
 			(at 22.86 138.43 0)
 			(effects
@@
 			)
 		)
-		(property "Footprint" "Button_Switch_SMD:SW_Push_1P1T_NO_6x6mm_H9.5mm"
+		(property "Footprint" "Button_Switch_THT:SW_PUSH_6mm_H9.5mm"
 			(at 33.02 60.96 0)
 			(effects
@@
 			)
 		)
-		(property "Datasheet" "~"
+		(property "Datasheet" "https://github.com/mael-lukas/2425_Projet2A_Animatronic/blob/main/Datasheets/Flex_Sensor_Datasheet_v2019a-3304101.pdf"
 			(at 114.3 138.43 0)
 			(effects
@@
 			)
 		)
-		(property "Datasheet" "~"
+		(property "Datasheet" "https://github.com/mael-lukas/2425_Projet2A_Animatronic/blob/main/Datasheets/Flex_Sensor_Datasheet_v2019a-3304101.pdf"
 			(at 68.58 138.43 0)
 			(effects

Commit message: pcb body & gant maj
Parts:
- added C10, C11, C12, C9: 100n, Capacitor_SMD:C_0402_1005Metric, symbol Device:C_Small
- added J3: Conn_01x02, symbol Connector_Generic:Conn_01x02
Connections:
- net +3.3V: now also C12.1, C9.2; no longer U2.8 (V+), U3.8 (V+)
- net GND: now also C10.2, C11.2, J3.2 (Pin_2); no longer U2.4 (V-), U3.4 (V-)
- new net: C11.1, U3.4 (V-)
- new net: C12.2, U3.8 (V+)
- new net: C9.1, U2.8 (V+)
- new net: C10.1, U2.4 (V-)
- new net +7.5V: J3.1 (Pin_1)
Other:
- note added: "batterie"

Commit message: PCB body & gant V3
Parts:
- removed C10, C11: 100n, Capacitor_SMD:C_0402_1005Metric, symbol Device:C_Small
- removed SW1: SW_SPST, Button_Switch_THT:SW_PUSH_6mm_H9.5mm, symbol Switch:SW_SPST
- added Flex1neg1, Flex1pos1, Flex2neg1, Flex2pos1, Flex3neg1, Flex3pos1: TestPoint, TestPoint:TestPoint_Pad_D1.5mm, symbol Connector:TestPoint
- added unit 2 of U3
- J3: footprint (none) -> Connector_JST:JST_EH_B2B-EH-A_1x02_P2.50mm_Vertical
Connections:
- net +7.5V is gone; now on net +5V: J3.1 (Pin_1)
- net +3.3V: now also R13.1, R14.1, U2.8 (V+), U3.8 (V+)
- net +5V: no longer R13.1, R14.1
- net GND: now also C12.2, C9.1, U2.4 (V-), U3.4 (V-), U3.5 (+), U3.6 (-)
- net at R3.2, R4.1, U2.3 (+): now also Flex1pos1.1
- net at R1.1, R2.1, U2.2 (-): now also Flex1neg1.1
- net at R10.1, R9.2, U3.3 (+): now also Flex3pos1.1
- net at R7.1, R8.1, U2.6 (-): now also Flex2neg1.1
- net at R5.2, R6.1, U2.5 (+): now also Flex2pos1.1
- net at R11.1, R12.1, U3.2 (-): now also Flex3neg1.1
- no-connect marks 19 -> 20
Other:
- moved on the sheet: C12, C9
